File: sensor.kicad_sch (KiCad schematic)
At the start: 64 parts, among them J1 10103594-0001LF, J2 , J4 , J5 , Q1 SI7423DN-T1-E3, U1 SN74LVC1G14DBV, U2 MAX17260SETD+, U3 MCP73831-2-OT, U4 STM32WB55xx, U5 MASWSS0115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

Commit message: First full draft
Connections:
- net PB5 is gone; now on net ENABLE_5V: U4.45 (PB5)
- net +3.3V: now also J4.7 (Pin_7); no longer J5.3 (Pin_3)
- net +5V: now also J5.12 (Pin_12)
- net ADC: now also J5.2 (Pin_2); no longer J5.1 (Pin_1)
- net ENABLE_5V: no longer U4.42 (PA15)
- net GND: now also J5.1 (Pin_1); no longer J5.10 (Pin_10), J5.12 (Pin_12)
- net LPUART1_RX: now also J5.7 (Pin_7); no longer J5.8 (Pin_8)
- net LPUART1_TX: now also J5.8 (Pin_8); no longer J5.9 (Pin_9)
- net NRST: now also J4.12 (Pin_12); no longer J4.7 (Pin_7)
- net PA0: now also J5.9 (Pin_9)
- net PB9: now also J5.10 (Pin_10); no longer J5.2 (Pin_2)
- net SPI1_MISO: now also J5.4 (Pin_4); no longer J5.5 (Pin_5)
- net SPI1_MOSI: now also J5.3 (Pin_3); no longer J5.4 (Pin_4)
- net SPI1_NSS: now also J5.6 (Pin_6); no longer J5.7 (Pin_7)
- net SPI1_SCK: now also J5.5 (Pin_5); no longer J5.6 (Pin_6)
- net SWCLK: now also J4.10 (Pin_10); no longer J4.9 (Pin_9)
- net SWDIO: now also J4.9 (Pin_9); no longer J4.8 (Pin_8)
- net SWO: now also J4.11 (Pin_11); no longer J4.10 (Pin_10)
- net PE4: now reaches U4.30 (PE4)
- net PE4: now also J4.5 (Pin_5)
- net ~{CHRG} renamed PA10
- net PA10: now also J4.8 (Pin_8)
- new net PA15: U4.42 (PA15)
Other:
- moved on the sheet: J4, J5

Commit message: Added I2C ports, rev2
Parts:
- added R5, R7: 1k, Resistor_SMD:R_0402_1005Metric, symbol Device:R
- added TP1, TP2, TP3, TP4, TP5, TP6, TP7: TestPoint, TestPoint:TestPoint_Pad_D1.0mm, symbol Connector:TestPoint
Connections:
- net PB0 is gone; now on net PB9: J4.3 (Pin_3)
- net PB8 is gone; now on net PA0: J4.2 (Pin_2)
- net +3.3V: now also R5.1, R7.1, TP2.1
- net +5V: now also TP4.1
- net +BATT: now also TP6.1
- net ANT_SEL: now also TP5.1
- net BAT_SENSE: now also TP3.1
- net I2C_SCL: now also J5.10 (Pin_10), R5.2
- net I2C_SDA: now also J5.9 (Pin_9), R7.2
- net PA0: no longer J5.9 (Pin_9)
- net PB9: no longer J5.10 (Pin_10)
- net VBUS: now also TP1.1
- net VDD: now also TP7.1
- net ~{FAULT}: no longer names the net of U4.44 (PB4)
- no-connect marks 5 -> 7

Commit message: Update
Parts:
- C4: MPN LMK063BBJ474KPLF -> CL10B474KO8NNND
Changed lines of the file:
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@@
       (effects (font (size 1.27 1.27)) hide)
     )
-    (property "MPN" "LMK063BBJ474KPLF" (id 4) (at 59.69 95.25 0)
+    (property "MPN" "CL10B474KO8NNND" (id 4) (at 59.69 95.25 0)
       (effects (font (size 1.27 1.27)) hide)
     )
